File: kicad/sp_et6/sp_et6.kicad_sch (KiCad schematic)
At the start: 125 parts, among them SW1 SW_PUSH, SW10 SW_PUSH, SW11 SW_PUSH, SW12 SW_PUSH, SW13 SW_PUSH, SW14 SW_PUSH, SW15 SW_PUSH, SW16 SW_PUSH, SW17 SW_PUSH, SW18 SW_PUSH, SW19 SW_PUSH, SW2 SW_PUSH, SW20 SW_PUSH, SW21 SW_PUSH, SW22 SW_PUSH, SW23 SW_PUSH, SW24 SW_PUSH, SW25 SW_PUSH, SW26 SW_PUSH, SW27 SW_PUSH, SW28 SW_PUSH, SW29 SW_PUSH, SW3 SW_PUSH, SW30 SW_PUSH, SW31 SW_PUSH, SW32 SW_PUSH, SW33 SW_PUSH, SW34 SW_PUSH, SW35 SW_PUSH, SW36 SW_PUSH, SW37 SW_PUSH, SW38 SW_PUSH, SW39 SW_PUSH, SW4 SW_PUSH, SW40 SW_PUSH, SW41 SW_PUSH, SW42 SW_PUSH, SW43 SW_PUSH, SW44 SW_PUSH, SW45 SW_PUSH, SW46 SW_PUSH, SW5 SW_PUSH, SW6 SW_PUSH, SW7 SW_PUSH, SW8 SW_PUSH, SW9 SW_PUSH, U2 PMW3610

Commit message: update sch
Parts:
- removed D35, D75: D, symbol Device:D
Connections:
- net pin6: now also D29.2 (A), D34.2 (A), D46.2 (A), D66.2 (A), SW21.1, SW22.1, SW23.1, SW27.1, SW31.1, SW35.1
Other:
- moved on the sheet: D12, D19, D63, D64

Commit message: kicad update
Other:
- note added: "RC(4,3)"
- note added: "RC(4,9)"
- note added: "RC(5,0)"
- note added: "RC(5,1)"
- note added: "RC(5,2)"
- note added: "RC(5,3)"
- note added: "RC(5,6)"
- note added: "RC(5,7)"
- note added: "RC(5,8)"
- note added: "RC(5,9)"
- note removed: "RC(0,11)"
- note removed: "RC(0,5)"
- note removed: "RC(1,11)"
- note removed: "RC(1,5)"
- note removed: "RC(2,11)"
- note removed: "RC(2,5)"
- note removed: "RC(3,10)"
- note removed: "RC(3,11)"
- note removed: "RC(3,4)"
- note removed: "RC(3,5)"
